File: circuit/Frank-Synced-BLDC-ESC.brd (EAGLE design)
At the start: 48.3 x 25.4 mm, 57 parts, among them IC1 Vreg +5V, Q1 PMOS-DPAK, Q2 NMOS-DPAK, Q4 PMOS-DPAK, Q5 NMOS-DPAK, Q7 PMOS-DPAK, Q8 NMOS-DPAK, U1 ATMEGA168MLF, U2 OSC-16MHz

Commit message: branch uses 2.5 x 2 mm sized +3.3V powered oscillator instead
Parts:
- added C11: 100n, Frank-Synced-BLDC-ESC:0603-CAP
- added IC3: Vreg +3V3, Frank-Synced-BLDC-ESC:SOT23-3
- C7: value 100n -> 1u
- U2: device Frank-Synced-BLDC-ESC:CRYSTAL-OSC-SMD-5X3 -> Frank-Synced-BLDC-ESC:OSCILLATOR-2.5X2
- moved C7 10.4 mm to (4.51, 1.91)
- moved C6 3.07 mm to (6.41, 1.91), turned to 270 degrees
- moved U2 1.20 mm to (8.76, 1.78)
- moved SJ3 0.84 mm to (4.91, 9.31), turned to 0 degrees
- moved SJ2 0.26 mm to (6.54, 4.83)
Connections:
- removed net N$25: C6.1, SJ2.1, U2.1, U2.4
- new net 3.3V: C6.1, IC3.2, U2.1, U2.4
- new net N$9: C7.1, IC3.3, SJ2.1
- net GND: now also C11.1, C7.2, IC3.1; no longer C7.1
- net RESET: now also C11.2; no longer C7.2
Routing:
- net N$25: track 8.13 -> 0.00 mm, vias 1 -> 0
- net 3.3V: track 0.00 -> 7.08 mm
- net N$9: track 0.00 -> 5.45 mm, vias 0 -> 1
- net TXD: track 10.2 -> 10.8 mm
- net GATE_N-C: track 32.8 -> 32.2 mm
- net GND: vias 25 -> 27
